File: KiCad/rokko_touch/mathrax-touch.kicad_pcb (KiCad board)
At the start: 2 copper layers, 350 x 18 mm, 31 parts

Commit message: update
Parts:
- moved PSOC4 78.0 mm to (73.7, 149.7)
- moved U$27 78.0 mm to (97.3, 143.9)
- moved C1 78.0 mm to (59.2, 152.0)
- moved C2 78.0 mm to (65.7, 154.5)
- moved C3 78.0 mm to (65.7, 152.0)
- moved C4 78.0 mm to (65.7, 144.5)
- moved C5 78.0 mm to (65.7, 142.0)
- moved C6 78.0 mm to (65.7, 139.5)
- moved F1 78.0 mm to (52.7, 150.5)
- moved LED0 78.0 mm to (66.2, 147.0)
- moved R1 78.0 mm to (66.7, 149.5)
- moved RS485 78.0 mm to (52.7, 143.5)
- moved U$1 78.0 mm to (74.2, 139.7)
- moved U$11 78.0 mm to (46.2, 147.0)
- moved U$13 78.0 mm to (60.2, 147.0)
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